File: lightsounds.kicad_sch (KiCad schematic)
At the start: 24 parts, among them J2 Conn_01x03_Female, T1 AO3400A, T2 AO3400A, T6 AO3400A

Commit message: 1.4.1 schematic update
Parts:
- EN1, boot1: symbol Connector:Conn_01x02_Female -> Connector:Conn_01x02_Socket
- EStop1, EStop2, J2, R-G-LED1: symbol Connector:Conn_01x03_Female -> Connector:Conn_01x03_Socket
Changed lines of the file:
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@@
 		)
 		(property "Datasheet" "http://www.aosmd.com/pdfs/datasheet/AO3400A.pdf"
-			(at 78.74 172.72 0)
-			(effects
-				(font
-					(size 1.27 1.27)
-				)
-				(justify left)
-				(hide yes)
-			)
-		)
-		(property "Description" ""
+			(at 74.93 177.8 0)
+			(effects
+				(font
+					(size 1.27 1.27)
+				)
+				(justify left)
+				(hide yes)
+			)
+		)
+		(property "Description" "30V Vds, 5.7A Id, N-Channel MOSFET, SOT-23"
 			(at 78.74 172.72 0)
 			(effects
@@
 			)
 		)
-		(property "Description" ""
+		(property "Description" "Power symbol creates a global label with name \"GND\" , ground"
 			(at 198.12 95.25 0)
 			(effects
@@
 	)
 	(symbol
-		(lib_id "Connector:Conn_01x02_Female")
+		(lib_id "Connector:Conn_01x02_Socket")
 		(at 104.14 67.31 0)
 		(unit 1)
@@
 			)
 		)
-		(property "Description" ""
+		(property "Description" "Generic connector, single row, 01x02, script generated"
 			(at 104.14 67.31 0)
 			(effects
@@
 	)
 	(symbol
-		(lib_name "+3.3V_1")
 		(lib_id "power:+3.3V")
 		(at 68.58 123.19 0)
@@
 			)
 		)
-		(property "Description" ""
+		(property "Description" "Power symbol creates a global label with name \"+3.3V\""
 			(at 68.58 123.19 0)
 			(effects
@@
 			)
 		)
-		(property "Description" ""
+		(property "Description" "Power symbol creates a global label with name \"GND\" , ground"
 			(at 66.04 74.93 0)
 			(effects
@@
 			)
 		)
-		(property "Description" ""
+		(property "Description" "Buzzer, polarized"
 			(at 200.66 72.39 0)
 			(effects
@@
 	)
 	(symbol
-		(lib_id "Connector:Conn_01x03_Female")
+		(lib_id "Connector:Conn_01x03_Socket")
 		(at 186.69 143.51 0)
 		(mirror x)
@@
 			)
 		)
-		(property "Description" ""
+		(property "Description" "Generic connector, single row, 01x03, script generated"
 			(at 186.69 143.51 0)
 			(effects
@@
 			)
 		)
-		(property "Description" ""
+		(property "Description" "Power symbol creates a global label with name \"GND\" , ground"
 			(at 91.44 135.89 0)
 			(effects
@@
 	)
 	(symbol
-		(lib_id "Connector:Conn_01x03_Female")
+		(lib_id "Connector:Conn_01x03_Socket")
 		(at 193.04 143.51 180)
 		(unit 1)
@@
 			)
 		)
-		(property "Description" ""
+		(property "Description" "Generic connector, single row, 01x03, script generated"
 			(at 193.04 143.51 0)
 			(effects
@@
 			)
 		)
-		(property "Description" ""
+		(property "Description" "Power symbol creates a global label with name \"GND\" , ground"
 			(at 102.87 179.07 0)
 			(effects
@@
 		)
 		(property "Datasheet" "http://www.aosmd.com/pdfs/datasheet/AO3400A.pdf"
-			(at 78.74 129.54 0)
-			(effects
-				(font
-					(size 1.27 1.27)
-				)
-				(justify left)
-				(hide yes)
-			)
-		)
-		(property "Description" ""
+			(at 74.93 134.62 0)
+			(effects
+				(font
+					(size 1.27 1.27)
+				)
+				(justify left)
+				(hide yes)
+			)
+		)
+		(property "Description" "30V Vds, 5.7A Id, N-Channel MOSFET, SOT-23"
 			(at 78.74 129.54 0)
 			(effects
@@
 	)
 	(symbol
-		(lib_name "+3.3V_1")
 		(lib_id "power:+3.3V")
 		(at 68.58 166.37 0)
@@
 			)
 		)
-		(property "Description" ""
+		(property "Description" "Power symbol creates a global label with name \"+3.3V\""
 			(at 68.58 166.37 0)
 			(effects
@@
 	)
 	(symbol
-		(lib_id "Connector:Conn_01x03_Female")
+		(lib_id "Connector:Conn_01x03_Socket")
 		(at 109.22 175.26 0)
 		(mirror x)
@@
 			)
 		)
-		(property "Description" ""
+		(property "Description" "Generic connector, single row, 01x03, script generated"
 			(at 109.22 175.26 0)
 			(effects
@@
 			)
 		)
-		(property "Description" ""
+		(property "Description" "Power symbol creates a global label with name \"+5V\""
 			(at 198.12 67.31 0)
 			(effects
@@
 			)
 		)
-		(property "Description" ""
+		(property "Description" "Power symbol creates a global label with name \"GND\" , ground"
 			(at 99.06 74.93 0)
 			(effects
@@
 	)
 	(symbol
-		(lib_id "Connector:Conn_01x02_Female")
+		(lib_id "Connector:Conn_01x02_Socket")
 		(at 71.12 67.31 0)
 		(unit 1)
@@
 			)
 		)
-		(property "Description" ""
+		(property "Description" "Generic connector, single row, 01x02, script generated"
 			(at 71.12 67.31 0)
 			(effects
@@
 			)
 		)
-		(property "Description" ""
+		(property "Description" "Power symbol creates a global label with name \"+5V\""
 			(at 91.44 166.37 0)
 			(effects
@@
 			)
 		)
-		(property "Description" ""
+		(property "Description" "Power symbol creates a global label with name \"+5V\""
 			(at 91.44 123.19 0)
 			(effects
@@
 		)
 		(property "Datasheet" "http://www.aosmd.com/pdfs/datasheet/AO3400A.pdf"
-			(at 195.58 83.82 0)
-			(effects
-				(font
-					(size 1.27 1.27)
-				)
-				(justify left)
-				(hide yes)
-			)
-		)
-		(property "Description" ""
+			(at 200.66 87.63 0)
+			(effects
+				(font
+					(size 1.27 1.27)
+				)
+				(justify left)
+				(hide yes)
+			)
+		)
+		(property "Description" "30V Vds, 5.7A Id, N-Channel MOSFET, SOT-23"
 			(at 195.58 83.82 0)
 			(effects
@@
 	)
 	(symbol
-		(lib_id "Connector:Conn_01x03_Female")
+		(lib_id "Connector:Conn_01x03_Socket")
 		(at 106.68 132.08 0)
 		(mirror x)
@@
 			)
 		)
-		(property "Description" ""
+		(property "Description" "Generic connector, single row, 01x03, script generated"
 			(at 106.68 132.08 0)
 			(effects
@@
 			)
 		)
-		(property "Description" ""
+		(property "Description" "Power symbol creates a global label with name \"GND\" , ground"
 			(at 160.02 144.78 0)
 			(effects

Commit message: update reference values for better ibom
Parts:
- renumbered D1 to D10, J2 to J100, EStop1 to J13, EStop2 to J14, R-G-LED1 to J15, boot1 to J18, EN1 to J19, R34 to R30, R35 to R31, T6 to T5
Other:
- note added: "E-Stop1"
- note added: "E-Stop2"
Changed lines of the file:
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@@
+		)
+	)
+	(text "E-Stop1"
+		(exclude_from_sim no)
+		(at 108.712 128.27 0)
+		(effects
+			(font
+				(size 2 2)
+				(thickness 0.4)
+				(bold yes)
+			)
+			(justify left bottom)
 		)
 	)
@@
 			)
 			(justify right bottom)
+		)
+	)
+	(text "E-Stop2"
+		(exclude_from_sim no)
+		(at 110.236 171.196 0)
+		(effects
+			(font
+				(size 2 2)
+				(thickness 0.4)
+				(bold yes)
+			)
+			(justify left bottom)
 		)
 	)
@@
 		(on_board yes)
 		(dnp no)
-		(property "Reference" "T6"
+		(property "Reference" "T5"
 			(at 80.01 179.07 0)
 			(effects
@@
 			(project "wing-combo"
 				(path "/586efc0f-7de2-49a7-ac21-ecfef2f716d6/3f0e9b91-fe15-47d5-84d6-aa71b368b91e/cdc711b4-3986-4d05-ace8-22e18ebb4f7d"
-					(reference "T6")
+					(reference "T5")
 					(unit 1)
 				)
@@
 		(on_board yes)
 		(dnp no)
-		(property "Reference" "EN1"
+		(property "Reference" "J19"
 			(at 105.41 67.3099 0)
 			(effects
@@
 			(project "wing-combo"
 				(path "/586efc0f-7de2-49a7-ac21-ecfef2f716d6/3f0e9b91-fe15-47d5-84d6-aa71b368b91e/cdc711b4-3986-4d05-ace8-22e18ebb4f7d"
-					(reference "EN1")
+					(reference "J19")
 					(unit 1)
 				)
@@
 		(dnp no)
 		(fields_autoplaced yes)
-		(property "Reference" "D1"
+		(property "Reference" "D10"
 			(at 210.7565 133.35 0)
 			(effects
@@
 			(project "wing-combo"
 				(path "/586efc0f-7de2-49a7-ac21-ecfef2f716d6/3f0e9b91-fe15-47d5-84d6-aa71b368b91e/cdc711b4-3986-4d05-ace8-22e18ebb4f7d"
-					(reference "D1")
+					(reference "D10")
 					(unit 1)
 				)
@@
 		(on_board yes)
 		(dnp no)
-		(property "Reference" "R-G-LED1"
+		(property "Reference" "J15"
 			(at 181.864 138.43 0)
 			(effects
@@
 			(project "wing-combo"
 				(path "/586efc0f-7de2-49a7-ac21-ecfef2f716d6/3f0e9b91-fe15-47d5-84d6-aa71b368b91e/cdc711b4-3986-4d05-ace8-22e18ebb4f7d"
-					(reference "R-G-LED1")
+					(reference "J15")
 					(unit 1)
 				)
@@
 		(on_board no)
 		(dnp no)
-		(property "Reference" "J2"
+		(property "Reference" "J100"
 			(at 194.31 138.43 90)
 			(effects
@@
 			(project "wing-combo"
 				(path "/586efc0f-7de2-49a7-ac21-ecfef2f716d6/3f0e9b91-fe15-47d5-84d6-aa71b368b91e/cdc711b4-3986-4d05-ace8-22e18ebb4f7d"
-					(reference "J2")
+					(reference "J100")
 					(unit 1)
 				)
@@
 		(on_board yes)
 		(dnp no)
-		(property "Reference" "EStop2"
+		(property "Reference" "J14"
 			(at 111.76 176.53 0)
 			(effects
@@
 			(project "wing-combo"
 				(path "/586efc0f-7de2-49a7-ac21-ecfef2f716d6/3f0e9b91-fe15-47d5-84d6-aa71b368b91e/cdc711b4-3986-4d05-ace8-22e18ebb4f7d"
-					(reference "EStop2")
+					(reference "J14")
 					(unit 1)
 				)
@@
 		(on_board yes)
 		(dnp no)
-		(property "Reference" "R34"
+		(property "Reference" "R30"
 			(at 63.5 168.91 0)
 			(effects
@@
 			(project "wing-combo"
 				(path "/586efc0f-7de2-49a7-ac21-ecfef2f716d6/3f0e9b91-fe15-47d5-84d6-aa71b368b91e/cdc711b4-3986-4d05-ace8-22e18ebb4f7d"
-					(reference "R34")
+					(reference "R30")
 					(unit 1)
 				)
@@
 		(on_board yes)
 		(dnp no)
-		(property "Reference" "R35"
+		(property "Reference" "R31"
 			(at 83.82 168.91 0)
 			(effects
@@
 			(project "wing-combo"
 				(path "/586efc0f-7de2-49a7-ac21-ecfef2f716d6/3f0e9b91-fe15-47d5-84d6-aa71b368b91e/cdc711b4-3986-4d05-ace8-22e18ebb4f7d"
-					(reference "R35")
+					(reference "R31")
 					(unit 1)
 				)
@@
 		(on_board yes)
 		(dnp no)
-		(property "Reference" "boot1"
+		(property "Reference" "J18"
 			(at 72.39 67.3099 0)
 			(effects
@@
 			(project "wing-combo"
 				(path "/586efc0f-7de2-49a7-ac21-ecfef2f716d6/3f0e9b91-fe15-47d5-84d6-aa71b368b91e/cdc711b4-3986-4d05-ace8-22e18ebb4f7d"
-					(reference "boot1")
+					(reference "J18")
 					(unit 1)
 				)
@@
 		(on_board yes)
 		(dnp no)
-		(property "Reference" "EStop1"
+		(property "Reference" "J13"
 			(at 109.22 130.81 0)
 			(effects
@@
 			(project "wing-combo"
 				(path "/586efc0f-7de2-49a7-ac21-ecfef2f716d6/3f0e9b91-fe15-47d5-84d6-aa71b368b91e/cdc711b4-3986-4d05-ace8-22e18ebb4f7d"
-					(reference "EStop1")
-					(unit 1)
-				)
+					(reference "J13")
+					(unit 1)
+				)
