File: stage1relays.kicad_sch (KiCad schematic)
At the start: 14 parts, among them T4 AO3400A, T7 AO3400A, U1 74HC02

Commit message: 1.4.1 schematic update
Parts:
- Bypass-1: symbol Connector:Conn_01x02_Female -> Connector:Conn_01x02_Socket
- renumbered T7 to T3
Other:
- note added: "The 'RESET' relay will break the electrical self-latch on the Stage 2 relay. Used as a way to auto shut-off the tool, in event of timeout. Bypass locks this relay 'OFF'"
- note added: "When `read-bypass` is ON this turns ON the `set` relay, but turns OFF the `reset` relay. By DeMorgan's Laws, that gives us the connections shown above. Note: the final NOT of the `reset` relay logic is in the relay itself."
- note added: "[!NOTE] We didn't want this to be able to automatically turn on a tool. The human intervention is a feature, not a bug. --- When this is 'ON' we commonly call the tool 'enabled' for use."
- note added: "check out our mock-up: tinkercad.com ~ sr-relays-bypass-74hc02-b1p3"
- note removed: "The 'RESET' relay will break the active self-latch on the Stage 2 relay. Used as a way to auto shut-off the tool, in event of timeout. Bypass locks this relay 'OFF'"
- note removed: "When `read-bypass` is ON this need to turn ON the `set` relay, but turn OFF the `reset` relay. By DeMorgan's Laws, that gives us the connections shown above. Note: the final NOT of the `reset` relay logic is in the relay itself."
- moved on the sheet: R40
Changed lines of the file:
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@@
 	(wire
 		(pts
-			(xy 177.8 97.79) (xy 177.8 101.6)
-		)
-		(stroke
-			(width 0)
-			(type default)
-		)
-	)
-	(wire
-		(pts
 			(xy 57.15 74.93) (xy 57.15 77.47)
 		)
@@
 	(wire
 		(pts
+			(xy 86.36 196.85) (xy 86.36 194.31)
+		)
+		(stroke
+			(width 0)
+			(type default)
+		)
+	)
+	(wire
+		(pts
 			(xy 170.18 92.71) (xy 161.29 92.71)
 		)
@@
 	(wire
 		(pts
-			(xy 177.8 74.93) (xy 177.8 77.47)
+			(xy 91.44 189.23) (xy 86.36 189.23)
 		)
 		(stroke
@@
 	(wire
 		(pts
-			(xy 161.29 81.28) (xy 161.29 77.47)
+			(xy 177.8 74.93) (xy 177.8 77.47)
 		)
 		(stroke
@@
 	(wire
 		(pts
-			(xy 185.42 97.79) (xy 185.42 101.6)
+			(xy 161.29 81.28) (xy 161.29 77.47)
 		)
 		(stroke
@@
 	(wire
 		(pts
+			(xy 86.36 189.23) (xy 86.36 191.77)
+		)
+		(stroke
+			(width 0)
+			(type default)
+		)
+	)
+	(wire
+		(pts
 			(xy 67.31 146.05) (xy 67.31 149.86)
 		)
@@
 	(wire
 		(pts
+			(xy 91.44 196.85) (xy 86.36 196.85)
+		)
+		(stroke
+			(width 0)
+			(type default)
+		)
+	)
+	(wire
+		(pts
 			(xy 67.31 146.05) (xy 71.12 146.05)
 		)
@@
 		)
 	)
-	(text "The 'RESET' relay will break the active self-latch on\nthe Stage 2 relay. Used as a way to auto shut-off the \ntool, in event of timeout. Bypass locks this relay 'OFF'"
+	(text "The 'RESET' relay will break the electrical self-latch on\nthe Stage 2 relay. Used as a way to auto shut-off the \ntool, in event of timeout. Bypass locks this relay 'OFF'"
 		(exclude_from_sim no)
 		(at 145.288 64.008 0)
@@
 		)
 	)
+	(text "check out our mock-up: tinkercad.com ~ sr-relays-bypass-74hc02-b1p3"
+		(exclude_from_sim no)
+		(at 160.782 157.226 0)
+		(effects
+			(font
+				(size 1.397 1.397)
+			)
+			(justify left bottom)
+			(href "https://www.tinkercad.com/things/2GyygmdKxWK-sr-relays-bypass-74hc02-b1p3")
+		)
+	)
 	(text "`set` relay: (ON if `set3v` is HIGH) OR (ON if read-bypass is HIGH [B-key is ON])\n`reset` relay: ON if read-bypass is LOW [B-key is OFF] AND reset3v is HIGH\n              --> else: `reset` relay is OFF [B-key can block `reset` relay]"
 		(exclude_from_sim no)
-		(at 160.782 161.29 0)
+		(at 160.782 165.608 0)
 		(effects
 			(font
@@
 		)
 	)
-	(text "When `read-bypass` is ON this need to turn ON the `set` relay, but turn OFF \nthe `reset` relay. By DeMorgan's Laws, that gives us the connections shown \nabove. Note: the final NOT of the `reset` relay logic is in the relay itself."
+	(text "[!NOTE] We didn't \nwant this to be able \nto automatically turn \non a tool. The human\nintervention is a \nfeature, not a bug.\n--- \nWhen this is 'ON' we\ncommonly call the tool\n'enabled' for use."
+		(exclude_from_sim no)
+		(at 100.584 99.314 0)
+		(effects
+			(font
+				(size 1.905 1.905)
+			)
+			(justify left bottom)
+		)
+	)
+	(text "When `read-bypass` is ON this turns ON the `set` relay, but turns OFF \nthe `reset` relay. By DeMorgan's Laws, that gives us the connections shown \nabove. Note: the final NOT of the `reset` relay logic is in the relay itself."
 		(exclude_from_sim no)
 		(at 160.782 152.908 0)
@@
 	)
 	(symbol
-		(lib_name "+3.3V_1")
 		(lib_id "power:+3.3V")
 		(at 64.77 142.24 0)
@@
 			)
 		)
-		(property "Description" ""
+		(property "Description" "Power symbol creates a global label with name \"+3.3V\""
 			(at 64.77 142.24 0)
 			(effects
@@
 			)
 		)
-		(property "Description" ""
+		(property "Description" "Power symbol creates a global label with name \"GND\" , ground"
 			(at 67.31 154.94 0)
 			(effects
@@
 	)
 	(symbol
-		(lib_name "+3.3V_1")
 		(lib_id "power:+3.3V")
 		(at 148.59 133.35 0)
@@
 			)
 		)
-		(property "Description" ""
+		(property "Description" "Power symbol creates a global label with name \"+3.3V\""
 			(at 148.59 133.35 0)
 			(effects
@@
 			)
 		)
-		(property "Description" ""
+		(property "Description" "Power symbol creates a global label with name \"GND\" , ground"
 			(at 123.19 195.58 0)
 			(effects
@@
 			)
 		)
-		(property "Description" ""
+		(property "Description" "Power symbol creates a global label with name \"+5V\""
 			(at 170.18 74.93 0)
 			(effects
@@
 			)
 		)
-		(property "Description" ""
+		(property "Description" "Power symbol creates a global label with name \"GND\" , ground"
 			(at 148.59 158.75 0)
 			(effects
@@
 			)
 		)
-		(property "Description" ""
+		(property "Description" "Power symbol creates a global label with name \"+5V\""
 			(at 123.19 181.61 0)
 			(effects
@@
 	(symbol
 		(lib_id "Device:R_US")
-		(at 181.61 97.79 270)
+		(at 181.61 101.6 270)
 		(mirror x)
 		(unit 1)
@@
 		(dnp no)
 		(property "Reference" "R40"
-			(at 181.61 93.218 90)
+			(at 181.61 97.028 90)
 			(effects
 				(font
@@
 		)
 		(property "Value" "1k"
-			(at 181.102 95.25 90)
+			(at 181.102 99.06 90)
 			(effects
 				(font
@@
 		)
 		(property "Footprint" "Resistor_SMD:R_0603_1608Metric"
-			(at 181.356 96.774 90)
+			(at 181.356 100.584 90)
 			(effects
 				(font
@@
 		)
 		(property "Datasheet" "~"
-			(at 181.61 97.79 0)
+			(at 181.61 101.6 0)
 			(effects
 				(font
@@
 		)
 		(property "Description" ""
-			(at 181.61 97.79 0)
+			(at 181.61 101.6 0)
 			(effects
 				(font
@@
 		)
 		(property "JLCPCB Part #" "C21190"
-			(at 181.61 97.79 90)
+			(at 181.61 101.6 90)
 			(effects
 				(font
@@
 	)
 	(symbol
-		(lib_id "Connector:Conn_01x02_Female")
+		(lib_id "Connector:Conn_01x02_Socket")
 		(at 76.2 146.05 0)
 		(mirror x)
@@
 			)
 		)
-		(property "Description" ""
+		(property "Description" "Generic connector, single row, 01x02, script generated"
 			(at 76.2 146.05 0)
 			(effects
@@
 	(symbol
 		(lib_id "power:GND")
-		(at 86.36 194.31 0)
+		(at 91.44 196.85 0)
 		(unit 1)
 		(exclude_from_sim no)
@@
 		(fields_autoplaced yes)
 		(property "Reference" "#PWR0160"
-			(at 86.36 200.66 0)
+			(at 91.44 203.2 0)
 			(effects
 				(font
@@
 		)
 		(property "Value" "GND"
-			(at 86.36 199.39 0)
+			(at 91.44 201.93 0)
 			(effects
 				(font
@@
 		)
 		(property "Footprint" ""
-			(at 86.36 194.31 0)
+			(at 91.44 196.85 0)
 			(effects
 				(font
@@
 		)
 		(property "Datasheet" ""
-			(at 86.36 194.31 0)
+			(at 91.44 196.85 0)
 			(effects
 				(font
@@
 			)
 		)
-		(property "Description" ""
-			(at 86.36 194.31 0)
+		(property "Description" "Power symbol creates a global label with name \"GND\" , ground"
+			(at 91.44 196.85 0)
 			(effects
 				(font
@@
 			)
 		)
-		(property "Description" ""
+		(property "Description" "Power symbol creates a global label with name \"GND\" , ground"
 			(at 57.15 114.3 0)
 			(effects
@@
 		(on_board yes)
 		(dnp no)
-		(property "Reference" "T7"
+		(property "Reference" "T3"
 			(at 61.976 103.886 0)
 			(effects
@@
 		)
 		(property "Datasheet" "http://www.aosmd.com/pdfs/datasheet/AO3400A.pdf"
-			(at 59.69 106.68 0)
+			(at 54.61 110.49 0)
 			(effects
 				(font
@@
 			)
 		)
-		(property "Description" ""
+		(property "Description" "30V Vds, 5.7A Id, N-Channel MOSFET, SOT-23"
 			(at 59.69 106.68 0)
 			(effects
@@
 			(project "wing-combo"
 				(path "/586efc0f-7de2-49a7-ac21-ecfef2f716d6/6f44f9bb-3a88-498d-9739-be3794f35f17/9191b819-8102-4422-9a84-62b3b85afe01"
-					(reference "T7")
+					(reference "T3")
 					(unit 1)
 				)
@@
 			)
 		)
-		(property "Description" ""
+		(property "Description" "Power symbol creates a global label with name \"+5V\""
 			(at 57.15 74.93 0)
 			(effects
@@
 			)
 		)
-		(property "Description" ""
+		(property "Description" "Power symbol creates a global label with name \"GND\" , ground"
 			(at 170.18 113.03 0)
 			(effects
@@
 		)
 		(property "Datasheet" "http://www.aosmd.com/pdfs/datasheet/AO3400A.pdf"
-			(at 172.72 101.6 0)
+			(at 167.64 105.41 0)
 			(effects
 				(font
@@
 			)
 		)
-		(property "Description" ""
+		(property "Description" "30V Vds, 5.7A Id, N-Channel MOSFET, SOT-23"
 			(at 172.72 101.6 0)
 			(effects
@@
 	(symbol
 		(lib_id "power:+5V")
-		(at 86.36 191.77 0)
+		(at 91.44 189.23 0)
 		(unit 1)
 		(exclude_from_sim no)
@@
 		(fields_autoplaced yes)
 		(property "Reference" "#PWR0161"
-			(at 86.36 195.58 0)
+			(at 91.44 193.04 0)
 			(effects
 				(font
@@
 		)
 		(property "Value" "+5V"
-			(at 86.36 186.69 0)
+			(at 91.44 184.15 0)
 			(effects
 				(font
@@
 		)
 		(property "Footprint" ""
-			(at 86.36 191.77 0)
+			(at 91.44 189.23 0)
 			(effects
 				(font
@@
 		)
 		(property "Datasheet" ""
-			(at 86.36 191.77 0)
+			(at 91.44 189.23 0)
 			(effects
 				(font
@@
 			)
 		)
-		(property "Description" ""
-			(at 86.36 191.77 0)
+		(property "Description" "Power symbol creates a global label with name \"+5V\""
+			(at 91.44 189.23 0)
 			(effects
 				(font

Commit message: update reference values for better ibom
Parts:
- renumbered D2 to D1, D3 to D2, D4 to D3, Bypass-1 to J10, R40 to R29
Changed lines of the file:
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@@
 		(dnp no)
 		(fields_autoplaced yes)
-		(property "Reference" "D2"
+		(property "Reference" "D1"
 			(at 127 192.0874 90)
 			(effects
@@
 			(project "wing-combo"
 				(path "/586efc0f-7de2-49a7-ac21-ecfef2f716d6/6f44f9bb-3a88-498d-9739-be3794f35f17/9191b819-8102-4422-9a84-62b3b85afe01"
-					(reference "D2")
+					(reference "D1")
 					(unit 1)
 				)
@@
 		(on_board yes)
 		(dnp no)
-		(property "Reference" "D3"
+		(property "Reference" "D2"
 			(at 48.26 81.28 90)
 			(effects
@@
 			(project "wing-combo"
 				(path "/586efc0f-7de2-49a7-ac21-ecfef2f716d6/6f44f9bb-3a88-498d-9739-be3794f35f17/9191b819-8102-4422-9a84-62b3b85afe01"
-					(reference "D3")
+					(reference "D2")
 					(unit 1)
 				)
@@
 		(on_board yes)
 		(dnp no)
-		(property "Reference" "R40"
+		(property "Reference" "R29"
 			(at 181.61 97.028 90)
 			(effects
@@
 			(project "wing-combo"
 				(path "/586efc0f-7de2-49a7-ac21-ecfef2f716d6/6f44f9bb-3a88-498d-9739-be3794f35f17/9191b819-8102-4422-9a84-62b3b85afe01"
-					(reference "R40")
+					(reference "R29")
 					(unit 1)
 				)
@@
 		(on_board yes)
 		(dnp no)
-		(property "Reference" "Bypass-1"
+		(property "Reference" "J10"
 			(at 72.898 140.716 0)
 			(effects
@@
 			(project "wing-combo"
 				(path "/586efc0f-7de2-49a7-ac21-ecfef2f716d6/6f44f9bb-3a88-498d-9739-be3794f35f17/9191b819-8102-4422-9a84-62b3b85afe01"
-					(reference "Bypass-1")
+					(reference "J10")
 					(unit 1)
 				)
@@
 		(on_board yes)
 		(dnp no)
-		(property "Reference" "D4"
+		(property "Reference" "D3"
 			(at 161.29 81.28 90)
 			(effects
@@
 			(project "wing-combo"
 				(path "/586efc0f-7de2-49a7-ac21-ecfef2f716d6/6f44f9bb-3a88-498d-9739-be3794f35f17/9191b819-8102-4422-9a84-62b3b85afe01"
-					(reference "D4")
-					(unit 1)
-				)
+					(reference "D3")
+					(unit 1)
+				)
