File: stage2relay.kicad_sch (KiCad schematic)
At the start: 5 parts, among them SW2 SW_Push, U4 PY14-02

Commit message: 1.4.1 schematic update
Connections:
- net Member-Green-Button-2: now also U4.9 (sw1-com); no longer U4.8 (sw4-no)
- net Stage3-Com: now also U4.12 (sw4-com); no longer U4.9 (sw1-com)
- net Stage3-NO: now also U4.8 (sw4-no); no longer U4.5 (sw1-no)
- net mains-fused-H/L1: now also U4.5 (sw1-no); no longer U4.12 (sw4-com)
Other:
- note added: "*If LED lamp us used, put resistor ABOVE the 'read' location."
- note added: "Both E-Stops (primary & aux): 1) shut off the tool at two 'layers' for redundancy 2) resets the active self-latch on the stage 2 relay 3) block green button use by member, locking out restarts All this works in redgular + bypass mode."
- note added: "Relay State Feedback to Microcontroller"
- note added: "S1-2 'reset' relay for timeout on tool"
- note added: "The firmware is more manageable if we sense the state of the relay (instead of infer the state from any electrical current readings). As long as 4PDT relay is used, microcontroller can sense relay state. DPDT versions of Omron MY relays will fit, but not connect this circuit."
- note added: "There are multiple variants of Omron's MY series relays, which allow for various coil voltage levels. ---> And this footprint also works with Omron's G2A relays, if there is ever a parts shortage..."
- note added: "This Estop is pysically coupled to 'Member-E-Stop-aux1' The EStop here (aux2) resets the active self-latch and also blocks the green button from working."
- note added: "This Estop is pysically coupled to 'Member-E-Stop-sw1' The EStop here (sw2) resets the active self-latch and also blocks the green button from working."
- note removed: "In this location, the E-Stop shuts off the tool and resets the active self-latch at the same time. and this works in bypass mode."
- note removed: "S1-2 relay for timeout on tool"
- note removed: "There are multiple variants of Omron's MY series relays, which allow for various voltage levels."
- note removed: "This Estop is linked to 'Member-E-Stop-sw1' The EStop here (sw2) resets the active self-latch and also blocks the green button from working."
- moved on the sheet: U4

Commit message: update reference values for better ibom
Parts:
- renumbered U4 to relay3
Changed lines of the file:
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@@
 		(on_board yes)
 		(dnp no)
-		(property "Reference" "U4"
+		(property "Reference" "relay3"
 			(at 87.376 134.366 0)
 			(effects
@@
 			(project ""
 				(path "/586efc0f-7de2-49a7-ac21-ecfef2f716d6/6f44f9bb-3a88-498d-9739-be3794f35f17/fd75559e-77bb-4f15-bd9f-e39243a04df3"
-					(reference "U4")
+					(reference "relay3")
 					(unit 1)
 				)
