File: microcontroller.kicad_sch (KiCad schematic)
At the start: 0 parts

Commit message: 1.4.1 schematic update
Other:
- note added: "This shows a component to represent the Adafruit Feather board, as it will be seated in place. However, the component itself is not included on the circuit board, instead seating into some breakout headers for easy replacement. This page is for reference only, not design. ---- Esperience implementing things like this on networks has taught us that it can be handy to be able to get a new device/MA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"
- note added: "This shows the relationships between all components running at 3.3VDC or 5VDC on the board. These are all on the 'low voltage' side of the board. These are all united in their service to the Adafruit Feather board. Thinkinc about this design as a whole. it is our past experience and makerspace spirit that guided us towards making this a Feather Wing rather than integrate the ESP32 on-board. If th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"
- note removed: "This shows a component to represent the Adafruit Feather board, as it will be seated in place. However, the component itself is not included on the circuit board, instead seating into some breakout headers for easy replacement. This page is for reference only, not design."
- note removed: "This shows the relationships between all components running at 3.3VDC or 5VDC on the board. These are all on the 'low voltage' side of the board. These are all united in their service to the Adafruit Feather board, but that board itself is removable (for ease of programming and switching out the controller, without needing to rewire the tools)."
Changed lines of the file:
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@@
 		(company "Corey Rice & MakeHaven")
 	)
-	(text "This shows the relationships between all components running at 3.3VDC or 5VDC on the board. \nThese are all on the 'low voltage' side of the board. These are all united in their service \nto the Adafruit Feather board, but that board itself is removable (for ease of programming \nand switching out the controller, without needing to rewire the tools). "
+	(text "This shows the relationships between all components running at 3.3VDC or 5VDC on the board. \nThese are all on the 'low voltage' side of the board. These are all united in their service \nto the Adafruit Feather board. Thinkinc about this design as a whole. it is our past experience\nand makerspace spirit that guided us towards making this a Feather Wing rather than integrate\nthe ESP32 on-board. If the microcontroller is removable, it is easier to program and you can \nreplace a 'problematic feather' for any reason, without needing to rewire the tools. "
 		(exclude_from_sim no)
-		(at 33.02 49.53 0)
+		(at 34.036 57.15 0)
 		(effects
 			(font
@@
 		)
 	)
-	(text "This shows a component to represent the \nAdafruit Feather board, as it will be \nseated in place. However, the component \nitself is not included on the circuit \nboard, instead seating into some breakout \nheaders for easy replacement. This page \nis for reference only, not design."
+	(text "This shows a component to represent the \nAdafruit Feather board, as it will be \nseated in place. However, the component \nitself is not included on the circuit \nboard, instead seating into some breakout \nheaders for easy replacement. This page \nis for reference only, not design.\n----\nEsperience implementing things like this on \nnetworks has taught us that it can be handy\nto be able to get a new device/MAC address \nwithout needing to rewire the entire 'box'\nthat connects to the tool."
 		(exclude_from_sim no)
-		(at 66.04 88.9 0)
+		(at 65.532 113.792 0)
 		(effects
 			(font
@@
 	(text "The ADE7953 is a high accuracy current, \nvoltage and power measurement chip that \ncommunicates with the ESP32 via I2C. \nThere are three 3.1mm audio jacks to \nenable connecting CT split-ring clamp \nsensors. These CT sensors can be \nclamped around the wires that run \npower to the tool, to monitor the \ncurrent and voltage draw throughout \nuse. Additionally, there are a number \nof jumpers that can be soldered to \nmodify the filtering circuits if \nnecessary. "
 		(exclude_from_sim no)
-		(at 175.26 105.41 0)
+		(at 175.26 113.03 0)
 		(effects
 			(font
@@
 	(text "ESP32 Core"
 		(exclude_from_sim no)
-		(at 33.02 67.31 0)
+		(at 33.02 74.93 0)
 		(effects
 			(font
@@
 	(text "ADE7953"
 		(exclude_from_sim no)
-		(at 143.51 66.04 0)
+		(at 143.51 73.66 0)
 		(effects
 			(font
@@
 	)
 	(sheet
-		(at 143.51 69.85)
+		(at 143.51 77.47)
 		(size 25.4 13.97)
 		(fields_autoplaced yes)
@@
 		)
 		(property "Sheetname" "ade7953"
-			(at 143.51 69.1384 0)
+			(at 143.51 76.7584 0)
 			(effects
 				(font
@@
 		)
 		(property "Sheetfile" "ade7953.kicad_sch"
-			(at 143.51 84.4046 0)
+			(at 143.51 92.0246 0)
 			(effects
 				(font
@@
 	)
 	(sheet
-		(at 34.29 71.12)
+		(at 34.29 78.74)
 		(size 25.4 13.97)
 		(fields_autoplaced yes)
@@
 		)
 		(property "Sheetname" "esp32core"
-			(at 34.29 70.4084 0)
+			(at 34.29 78.0284 0)
 			(effects
 				(font
@@
 		)
 		(property "Sheetfile" "esp32core.kicad_sch"
-			(at 34.29 85.6746 0)
+			(at 34.29 93.2946 0)
 			(effects
 				(font

Commit message: nearly ready
Other:
- added sheet usb-c-power-out (usb-c-power-out.kicad_sch)
- note added: "It is foreseeable that daughter baords will be added, and these connections allow for the ability to power them without needing a second AC/DC Power Supply. These are fused to not over-draw from the main baords/ uses."
- note added: "USB-C & Solder | Daughter Power"
Changed lines of the file:
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@@
 	(text "This shows a component to represent the \nAdafruit Feather board, as it will be \nseated in place. However, the component \nitself is not included on the circuit \nboard, instead seating into some breakout \nheaders for easy replacement. This page \nis for reference only, not design.\n----\nEsperience implementing things like this on \nnetworks has taught us that it can be handy\nto be able to get a new device/MAC address \nwithout needing to rewire the entire 'box'\nthat connects to the tool."
 		(exclude_from_sim no)
-		(at 65.532 113.792 0)
+		(at 68.072 106.172 0)
 		(effects
 			(font
@@
 	(text "Breakout Board Connections"
 		(exclude_from_sim no)
-		(at 33.02 128.27 0)
+		(at 35.56 120.65 0)
 		(effects
 			(font
@@
 	(text "These are the connections for I2C, SPI, and \nthe Feather headers. There is also a 3.3V \nlinear regulator to power these daughter \nboards, without placing more draw on the \nFeather's onboard linear regulator (this \nincludes powering the ADE7953).\n\nThere are also USB plugs to provide \naccess to 5VDC - this is primarily \nto power the Feaather, as they are \ndesigned to be powered this way or by\nbattery. The second USB port could power \nfuture independent e-ink displays, etc.\n"
 		(exclude_from_sim no)
-		(at 64.77 166.37 0)
+		(at 67.31 158.75 0)
 		(effects
 			(font
@@
 	(text "ESP32 Core"
 		(exclude_from_sim no)
-		(at 33.02 74.93 0)
-		(effects
-			(font
-				(size 3.5 3.5)
-				(bold yes)
+		(at 35.56 67.31 0)
+		(effects
+			(font
+				(size 3.5 3.5)
+				(bold yes)
+			)
+			(justify left bottom)
+		)
+	)
+	(text "USB-C & Solder | Daughter Power"
+		(exclude_from_sim no)
+		(at 35.052 174.752 0)
+		(effects
+			(font
+				(size 3.5 3.5)
+				(bold yes)
+			)
+			(justify left bottom)
+		)
+	)
+	(text "It is foreseeable that daughter baords will \nbe added, and these connections allow for \nthe ability to power them without needing\na second AC/DC Power Supply. These are fused\nto not over-draw from the main baords/ uses."
+		(exclude_from_sim no)
+		(at 72.136 191.77 0)
+		(effects
+			(font
+				(size 1.75 1.75)
 			)
 			(justify left bottom)
@@
 	)
 	(sheet
-		(at 34.29 78.74)
+		(at 36.83 71.12)
 		(size 25.4 13.97)
 		(fields_autoplaced yes)
@@
 		)
 		(property "Sheetname" "esp32core"
-			(at 34.29 78.0284 0)
+			(at 36.83 70.4084 0)
 			(effects
 				(font
@@
 		)
 		(property "Sheetfile" "esp32core.kicad_sch"
-			(at 34.29 93.2946 0)
+			(at 36.83 85.6746 0)
 			(effects
 				(font
@@
 	)
 	(sheet
-		(at 34.29 130.81)
+		(at 36.83 123.19)
 		(size 25.4 13.97)
 		(fields_autoplaced yes)
@@
 		)
 		(property "Sheetname" "breakoutboards"
-			(at 34.29 130.0984 0)
+			(at 36.83 122.4784 0)
 			(effects
 				(font
@@
 		)
 		(property "Sheetfile" "breakoutboards.kicad_sch"
-			(at 34.29 145.3646 0)
+			(at 36.83 137.7446 0)
 			(effects
 				(font
@@
 				)
 			)
+		)
+	)
+	(sheet
+		(at 36.83 177.8)
+		(size 25.4 13.97)
+		(fields_autoplaced yes)
+		(stroke
+			(width 0.1524)
+			(type solid)
+		)
+		(fill
+			(color 0 0 0 0.0000)
+		)
+		(property "Sheetname" "usb-c-power-out"
+			(at 36.83 177.0884 0)
+			(effects
+				(font
+					(size 1.27 1.27)
+				)
+				(justify left bottom)
+			)
+		)
+		(property "Sheetfile" "usb-c-power-out.kicad_sch"
+			(at 36.83 192.3546 0)
+			(effects
+				(font
+					(size 1.27 1.27)
+				)
+				(justify left top)
+			)
+		)
+		(instances
+			(project "wing-combo"
+				(path "/586efc0f-7de2-49a7-ac21-ecfef2f716d6/3f0e9b91-fe15-47d5-84d6-aa71b368b91e"
+					(page "11")
+				)
+			)
