File: usb-c-power-out.kicad_sch (KiCad schematic)
At the start: 11 parts, among them J8 USB_C_Receptacle_USB2.0_16P, J9 Conn_01x02_Female, Q1 PMOS, U4 LM393

Commit message: 5v binary current and cleanup
Other:
- note added: "Power-only USB"
- note added: "The Upstream-Facing Port (UFP) will supply 5.1k resistor(s) on at least one of the plug's `CC1` or `CC2` lines"
- note added: "This USB port only supplies power, not a data connection anywhere. If you remove JP24, this can power the feather [NOT advised]. The USB can power secondary microcontrollers (like for e-Ink)."
- note added: "This is a minimum-viable USB-C source. Connecting a USB-C device to this port will activate at least one comparator, and turn on power to the `VBUS` only after a connection is made. This behavior is called 'Cold Plugging' and is an expectation of USB-C Downside-Facing Ports (DFP). The fuse will limit the current to roughly 500mA, and trip if 1A is ever pulled from this device. This is another exp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"
- note added: "While it is not entirely clear how these will be used, they provide options for powering secondary daugher boards without needing to add a second AC/DC Power Supply unit to the tool-controller box. The easiest attachment is a USB-C source plug (technically a DFP) that is basically compliant with the proper USB-C specifications. Also, there is a pair of solderable holes that allow for a more-direc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"
- note removed: "Power-only USB out"
- note removed: "The Feather is powered via USB, by specification. These allow for short cables to supply 5V power. May be also used to power secondary microcontrollers (like for e-Ink)."
- note removed: "The Upside Facing Port (UFP) will supply 5.1k resistor(s) on at least one of the plug's `CC1` or `CC2` lines"
- note removed: "This is a minimum-viable USB-C source. Connecting a USB-C device to this port will activate at least one comparator, and turn on power to the `VBUS` only after a connection is made. This behavior is called 'Cold Plugging' and is an expectation of USB-C Downward Facing Ports (DFP). The fuse will limit the current to roughly 500mA, and trip if 1A is even pulled from this device. This is another exp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"
- note removed: "While it is not entirely clear how these will be used, they provide options for powering secondary daugher boards without needing to add a second AC/DC Power Supply unit to the tool-controller box. The easiest attachment is a USB-C source plug (technically a DFP) that is nearly compliant with the prper USB-C specifications. Also, there is a pair of solderable holes that allow for a more-direct co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"
- moved on the sheet: C24, J8, R36, R37, U4C

Commit message: close enough for 3D export
Other:
- note added: "The Upstream-Facing Port (UFP) will supply 5.1k resistor(s) on at least one of the plug's `CC1` or `CC2` lines (which is the expectation of the USB_C specifications). This brings the '+' input low, and activates the comparator to sink current."
- note added: "While it is not entirely clear how these will be used, they provide options for powering secondary daugher boards without needing to add a second AC/DC Power Supply unit to the tool-controller box. The easiest attachment is a USB-C source plug (technically a DFP) that is basically compliant with the proper USB-C specifications. Also, there is a pair of solderable holes that allow for a more direc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"
- note removed: "The Upstream-Facing Port (UFP) will supply 5.1k resistor(s) on at least one of the plug's `CC1` or `CC2` lines"
- note removed: "While it is not entirely clear how these will be used, they provide options for powering secondary daugher boards without needing to add a second AC/DC Power Supply unit to the tool-controller box. The easiest attachment is a USB-C source plug (technically a DFP) that is basically compliant with the proper USB-C specifications. Also, there is a pair of solderable holes that allow for a more-direc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"
- company: (none) -> Corey Rice / MakeHaven
Changed lines of the file:
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@@
 		(title "5V USB-C and Pins | Daughter Board Power")
 		(date "2025-10-04")
+		(company "Corey Rice / MakeHaven")
+		(comment 1 "Solderable connection also provided, still guarded by resettable fuse")
+		(comment 2 "Features Cold-Plugging with an LM393 and over current protection")
+		(comment 3 "Bare-minimum USB-C downside facing port")
 	)
 	(junction
@@
 		)
 	)
-	(text "While it is not entirely clear how these will be used, they provide options for powering secondary daugher boards\nwithout needing to add a second AC/DC Power Supply unit to the tool-controller box. The easiest attachment is a \nUSB-C source plug (technically a DFP) that is basically compliant with the proper USB-C specifications. Also, there is\na pair of solderable holes that allow for a more-direct connection to the 5V line, but are still guarded by the \nresettable fuse. Either of these could be used to add a panel-mount USB-C port, and then attach a second MCU for \nany number of purposes: we think an E-Ink display for machine status could be really helpful :)"
+	(text "While it is not entirely clear how these will be used, they provide options for powering secondary daugher boards\nwithout needing to add a second AC/DC Power Supply unit to the tool-controller box. The easiest attachment is a \nUSB-C source plug (technically a DFP) that is basically compliant with the proper USB-C specifications. Also, there is\na pair of solderable holes that allow for a more direct connection to the 5V line, but is still guarded by the shared\nresettable fuse. Either of these could be used to add a panel-mount USB-C port, and then attach a second MCU for \nany number of purposes: ==> We think an E-Ink display for machine status could be really helpful :)"
 		(exclude_from_sim no)
 		(at 35.052 40.894 0)
@@
 		)
 	)
-	(text "The Upstream-Facing Port (UFP) will supply 5.1k resistor(s) \non at least one of the plug's `CC1` or `CC2` lines"
-		(exclude_from_sim no)
-		(at 46.99 118.11 0)
-		(effects
-			(font
+	(text "The Upstream-Facing Port (UFP) will supply 5.1k resistor(s) \non at least one of the plug's `CC1` or `CC2` lines (which is\nthe expectation of the USB_C specifications). This brings the \n'+' input low, and activates the comparator to sink current."
+		(exclude_from_sim no)
+		(at 44.958 120.142 0)
+		(effects
+			(font
